Commit message: 单车修改

File: ros2_ws/src/my_robot/urdf/diffbot.urdf.xacro (robot description, xacro)
@@ -3,4 +3,11 @@
   <xacro:property name="wheel_radius" value="0.075"/>
   <xacro:property name="wheel_separation" value="0.32"/>
+  <!-- base_footprint 用于2D导航常见基座帧 -->
+  <link name="base_footprint"/>
+  <joint name="base_footprint_joint" type="fixed">
+    <parent link="base_footprint"/>
+    <child link="base_link"/>
+    <origin xyz="0 0 0" rpy="0 0 0"/>
+  </joint>
   <!-- Base Link (车体) -->
   <link name="base_link">
@@ -161,7 +168,4 @@
    <gazebo>
     <plugin name="joint_state_publisher" filename="libgazebo_ros_joint_state_publisher.so">
-      <ros>
-        <remapping>joint_states:=wheel_joint_states</remapping>
-      </ros>
       <update_rate>100</update_rate>
       <joint_name>left_wheel_joint</joint_name>

Commit message: 代码完整版带imu

File: ros2_ws/src/my_robot/urdf/diffbot.urdf.xacro (robot description, xacro)
@@ -6,6 +6,6 @@
   <link name="base_footprint"/>
   <joint name="base_footprint_joint" type="fixed">
-    <parent link="base_footprint"/>
-    <child link="base_link"/>
+    <parent link="base_link"/>
+    <child link="base_footprint"/>
     <origin xyz="0 0 0" rpy="0 0 0"/>
   </joint>
@@ -188,5 +188,5 @@
       <!-- limits -->
       <max_wheel_torque>40</max_wheel_torque>
-      <max_wheel_acceleration>12.0</max_wheel_acceleration>
+      <max_wheel_acceleration>18.0</max_wheel_acceleration>
       <!-- output -->
       <publish_odom>true</publish_odom>
@@ -265,4 +265,36 @@
     <origin xyz="0.2 0 0.08" rpy="0 0 0"/>
   </joint>
+  <!-- IMU (姿态稳定用) -->
+  <link name="imu_link">
+    <inertial>
+      <origin xyz="0 0 0" rpy="0 0 0"/>
+      <mass value="0.05"/>
+      <inertia ixx="1e-5" ixy="0" ixz="0" iyy="1e-5" iyz="0" izz="1e-5"/>
+    </inertial>
+    <visual>
+      <geometry>
+        <box size="0.02 0.02 0.01"/>
+      </geometry>
+      <material name="black"/>
+    </visual>
+  </link>
+  <joint name="imu_joint" type="fixed">
+    <parent link="base_link"/>
+    <child link="imu_link"/>
+    <origin xyz="0.0 0.0 0.12" rpy="0 0 0"/>
+  </joint>
+  <gazebo reference="imu_link">
+    <sensor name="imu_sensor" type="imu">
+      <always_on>true</always_on>
+      <update_rate>100</update_rate>
+      <visualize>false</visualize>
+      <plugin name="imu_controller" filename="libgazebo_ros_imu_sensor.so">
+        <ros>
+          <argument>~/out:=imu/data</argument>
+        </ros>
+        <frame_name>imu_link</frame_name>
+      </plugin>
+    </sensor>
+  </gazebo>
   <gazebo reference="camera_link">
     <material>Gazebo/Black</material>
